File: case/plates/top-plate-hybrid/top-plate-hybrid.kicad_pcb (KiCad board)
At the start: 2 copper layers, 103.9 x 80.6 mm, 0 parts

Commit message: small change
Routing:
- added copper zone on B.Cu, net (none)
- added copper zone on F.Cu, net (none)
- removed copper zone on B.Cu, net GND
- removed copper zone on F.Cu, net GND
Changed lines of the file:
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@@
 	)
 	(net 0 "")
-	(net 1 "GND")
 	(gr_circle
 		(center 74.609926 64.290043)
@@
 			(type solid)
 		)
-		(fill solid)
+		(fill none)
 		(layer "Edge.Cuts")
 	)
@@
 	)
 	(zone
-		(net 1)
-		(net_name "GND")
+		(net 0)
+		(net_name "")
 		(layers "F&B.Cu")
 		(hatch edge 0.5)
