File: case/plates/top-plate-hybrid/top-plate-hybrid.kicad_sch (KiCad schematic)
At the start: 0 parts

Commit message: Mcu cover (#7)
* more plates

* updated workflow

* mcu cover

* small change
Other:
- company: (none) -> Allen Choi
- title: VOID top plate hybrid -> VOID Top Plate Hybrid
Changed lines of the file:
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@@
 	(paper "A4")
 	(title_block
-		(title "VOID top plate hybrid")
+		(title "VOID Top Plate Hybrid")
 		(date "2024-11-17")
 		(rev "0.5.9")
+		(company "Allen Choi")
 	)
 	(sheet_instances
