File: case/plates/bottom-plate/bottom-plate.kicad_sch (KiCad schematic)
At the start: 0 parts

Commit message: Mcu cover (#7)
* more plates

* updated workflow

* mcu cover

* small change
Other:
- title: VOID bottom plate -> VOID Bottom Plate
Changed lines of the file:
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@@
 	(paper "A4")
 	(title_block
-		(title "VOID bottom plate")
+		(title "VOID Bottom Plate")
 		(date "2024-11-17")
 		(rev "0.5.9")
