File: chocolate/void-3x5-chocolate.kicad_pcb (KiCad board)
At the start: 2 copper layers, 140.5 x 112.5 mm, 82 parts, among them J1 USB_C_Receptacle_PowerOnly_6P, J2 Conn_01x02, J3 Conn_01x02, J4 Conn_01x03

Commit message: Quick fixes (#16)
* fix version

* updated PCB
Other:
- board text added: "VOID v0.6.1"
- board text removed: "VOID v0.6.0"

Commit message: updated kicad data
Parts:
- R1: footprint Resistor_SMD:R_0805_2012Metric_Pad1.20x1.40mm_HandSolder -> TB2086_SMD:R_0805_2012Metric_Pad1.20x1.40mm_HandSolder; moved to F.Cu
- R2: footprint Resistor_SMD:R_0805_2012Metric_Pad1.20x1.40mm_HandSolder -> TB2086_SMD:R_0805_2012Metric_Pad1.20x1.40mm_HandSolder
Connections:
- RSW1 pad MP: (no net) -> GND
