File: chocolate/void-3x5-chocolate.kicad_sch (KiCad schematic)
At the start: 80 parts, among them J1 Conn_01x02, J2 Conn_01x03_MountingPin, J3 Conn_01x02

Commit message: choc
Parts:
- MCU1: footprint TB2086_MISC:ProMicro-dn-rev-unrouted -> TB2086_MISC:ProMicro-dn-flipped-rev-unrouted
Changed lines of the file:
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@@
 			)
 		)
-		(property "Footprint" "TB2086_MISC:ProMicro-dn-rev-unrouted"
+		(property "Footprint" "TB2086_MISC:ProMicro-dn-flipped-rev-unrouted"
 			(at 62.992 63.5 0)
 			(effects

Commit message: Choc (#4)
* updated mcu footprint for choc

* added holes for oled window

* hybrid top plate

* added hybrid top plate
Parts:
- MCU1: footprint TB2086_MISC:ProMicro-dn-flipped-rev-unrouted -> TB2086_MISC:ProMicro-dn-rev-unrouted
Changed lines of the file:
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@@
 			)
 		)
-		(property "Footprint" "TB2086_MISC:ProMicro-dn-flipped-rev-unrouted"
+		(property "Footprint" "TB2086_MISC:ProMicro-dn-rev-unrouted"
 			(at 62.992 63.5 0)
 			(effects

Commit message: updated choc
Parts:
- removed J1, J3: Conn_01x02, TB2086_SMD:Molex_Pico-EZmate_78171-0002_1x02-1MP_P1.20mm_Vertical_rev, symbol Connector_Generic_MountingPin:Conn_01x02_MountingPin
- removed J2: Conn_01x03_MountingPin, TB2086_SMD:TE_0-1734839-5_1x05-1MP_P0.5mm_Horizontal_rev, symbol Connector_Generic_MountingPin:Conn_01x05_MountingPin
- removed TRRS1: MJ-4PP-9, TB2086_MISC:TRRS-PJ-320A-rev, symbol TB2086_MISC:MJ-4PP-9
- added J1: USB_C_Receptacle_PowerOnly_6P, TB2086_SMD:USB-20C-F-6C16_rev, symbol Connector:USB_C_Receptacle_PowerOnly_6P
- added J2: Conn_01x02, TB2086_SMD:JST_PH_S2B-PH-SM4-TB_1x02-1MP_P2.00mm_Horizontal_rev, symbol Connector_Generic_MountingPin:Conn_01x02_MountingPin
- added J3: Conn_01x02, TB2086_MISC:Pogopin_1x02_P2.54mm, symbol Connector_Generic:Conn_01x02
- added J4: Conn_01x03, TB2086_MISC:Pogopin_1x03_P2.54mm, symbol Connector_Generic:Conn_01x03
- added LOGO2: Logo_Open_Hardware_Small, TB2086_MISC:OSHW-Logo_5.7x6mm_SilkScreen_rev, symbol Graphic:Logo_Open_Hardware_Small
- added SW_SPDT2: SW_SPDT2, TB2086_SMD:SW_SPDT_PCM12, symbol Switch:SW_SPDT
- LOGO1: value Logo_Open_Hardware_Small -> Logo_Open_ErgoGen
- SW_SPDT1: value SW_SPDT -> SW_SPDT1; footprint TB2086_SMD:SW_SPDT_PCM12_reversible -> TB2086_SMD:SW_SPDT_PCM12
Connections:
- net BAT: now also J3.2 (Pin_2), SW_SPDT2.3 (C)
- net GND: now also J1.A12 (GND), J1.B12 (GND), J1.S1 (SHIELD), J2.1 (Pin_1), J2.MP (MountPin), J3.1 (Pin_1)
- net VCC: now also J1.A9 (VBUS), J1.B9 (VBUS)
- net at SW_SPDT1.2 (B): now also J2.2 (Pin_2), SW_SPDT2.2 (B)
- net at LED3.1 (K), LED4.1 (K): now also J4.3 (Pin_3)
- net at LED1.2 (A), LED2.2 (A), LED3.2 (A)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: now also J4.2 (Pin_2)
- net at LED1.1 (K), LED2.1 (K): now also J4.1 (Pin_1)
- net at JP3.2 (B): now also J1.A5 (CC1)
- net at JP2.2 (C): now also J1.B5 (CC2)
- no-connect marks 8 -> 9
Other:
- moved on the sheet: D10, D11, D12, D13, D14, D15, D4, D5, D6, D7, D8, D9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

Commit message: Quick fixes (#16)
* fix version

* updated PCB
Other:
- title: uniCorne Cherry -> VOID 3x5 Choc
Changed lines of the file:
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@@
 	(paper "A3")
 	(title_block
-		(title "uniCorne Cherry")
-		(date "2023-07-20")
-		(rev "0.9")
+		(title "VOID 3x5 Choc")
+		(date "2025-02-02")
+		(rev "0.6.1")
 		(company "Thunderbird2086")
 	)

Commit message: updated kicad data
Parts:
- R1, R2: footprint Resistor_SMD:R_0805_2012Metric_Pad1.20x1.40mm_HandSolder -> TB2086_SMD:R_0805_2012Metric_Pad1.20x1.40mm_HandSolder
Changed lines of the file:
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@@
 			)
 		)
-		(property "Footprint" "Resistor_SMD:R_0805_2012Metric_Pad1.20x1.40mm_HandSolder"
+		(property "Footprint" "TB2086_SMD:R_0805_2012Metric_Pad1.20x1.40mm_HandSolder"
 			(at 67.31 77.978 90)
 			(effects
@@
 			)
 		)
-		(property "Footprint" "Resistor_SMD:R_0805_2012Metric_Pad1.20x1.40mm_HandSolder"
+		(property "Footprint" "TB2086_SMD:R_0805_2012Metric_Pad1.20x1.40mm_HandSolder"
 			(at 67.31 68.707 90)
 			(effects
