File: hybrid-mx/void-3x5-hybrid-mx.kicad_pcb (KiCad board)
At the start: 2 copper layers, 140.5 x 112.5 mm, 82 parts, among them J1 USB_C_Receptacle_PowerOnly_6P, J2 Conn_01x02, J3 Conn_01x02, J4 Conn_01x03

Commit message: Quick fixes (#16)
* fix version

* updated PCB
Other:
- board text added: "VOID v0.6.1"
- board text removed: "VOID v0.6.0"

Commit message: updated kicad data
Connections:
- RSW1 pad MP: (no net) -> GND
