File: hybrid-mx/void-3x5-hybrid-mx.kicad_sch (KiCad schematic)
At the start: 80 parts, among them J1 Conn_01x02, J2 Conn_01x03_MountingPin, J3 Conn_01x02

Commit message: fixed bridge for hybrid-mx
Parts:
- S16, S17: value SW_CHOC_HS -> SW_MX_HS; footprint TB2086_KEYSWITCH:SW_choc_v1_v2_HS_1u_reversible -> TB2086_KEYSWITCH:SW_MX_HS_1u_reversible
- S18: value SW_CHOC_HS -> SW_MX_HS; footprint TB2086_KEYSWITCH:SW_choc_v1_v2_HS_1.5u_reversible -> TB2086_KEYSWITCH:SW_MX_HS_1.5u_reversible
Changed lines of the file:
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@@
 			)
 		)
-		(property "Value" "SW_CHOC_HS"
+		(property "Value" "SW_MX_HS"
 			(at 175.133 106.553 0)
 			(effects
@@
 			)
 		)
-		(property "Footprint" "TB2086_KEYSWITCH:SW_choc_v1_v2_HS_1u_reversible"
+		(property "Footprint" "TB2086_KEYSWITCH:SW_MX_HS_1u_reversible"
 			(at 170.942 106.172 0)
 			(effects
@@
 			)
 		)
-		(property "Value" "SW_CHOC_HS"
+		(property "Value" "SW_MX_HS"
 			(at 192.913 106.553 0)
 			(effects
@@
 			)
 		)
-		(property "Footprint" "TB2086_KEYSWITCH:SW_choc_v1_v2_HS_1u_reversible"
+		(property "Footprint" "TB2086_KEYSWITCH:SW_MX_HS_1u_reversible"
 			(at 188.722 106.172 0)
 			(effects
@@
 			)
 		)
-		(property "Value" "SW_CHOC_HS"
+		(property "Value" "SW_MX_HS"
 			(at 210.693 106.553 0)
 			(effects
@@
 			)
 		)
-		(property "Footprint" "TB2086_KEYSWITCH:SW_choc_v1_v2_HS_1.5u_reversible"
+		(property "Footprint" "TB2086_KEYSWITCH:SW_MX_HS_1.5u_reversible"
 			(at 206.502 106.172 0)
 			(effects

Commit message: Changed TRRS to USB-C connector (#14)
* usb-c mod for hybrid

* updated
  - submodule
  - ergogen yaml
  - schematic and pcb

* updated cherry-mx

usb-c for communication between left and right hand sides

* updated choc

* updated choc

* fixed corner

* void-choc

* ergogen
  - bottom plate
  - charger plate

* updated choc

* updated ergogen

* cherry-mx
* hybrid-mx

* updated ergogen for VOID Choc

* refreshed submodule

* updated ergogen yaml

* updated PCBs

* updated version
Parts:
- removed J2: Conn_01x03_MountingPin, TB2086_SMD:TE_0-1734839-5_1x05-1MP_P0.5mm_Horizontal_rev, symbol Connector_Generic_MountingPin:Conn_01x05_MountingPin
- removed J3: Conn_01x02, TB2086_SMD:Molex_Pico-EZmate_78171-0002_1x02-1MP_P1.20mm_Vertical_rev, symbol Connector_Generic_MountingPin:Conn_01x02_MountingPin
- removed TRRS1: MJ-4PP-9, TB2086_MISC:TRRS-PJ-320A-rev, symbol TB2086_MISC:MJ-4PP-9
- added J1: USB_C_Receptacle_PowerOnly_6P, TB2086_SMD:USB-20C-F-6C16_rev, symbol Connector:USB_C_Receptacle_PowerOnly_6P
- added J3: Conn_01x02, TB2086_MISC:Pogopin_1x02_P2.54mm, symbol Connector_Generic:Conn_01x02
- added J4: Conn_01x03, TB2086_MISC:Pogopin_1x03_P2.54mm, symbol Connector_Generic:Conn_01x03
- added LOGO2: Logo_Open_Hardware_Small, TB2086_MISC:OSHW-Logo_5.7x6mm_SilkScreen_rev, symbol Graphic:Logo_Open_Hardware_Small
- added SW_SPDT1: SW_SPDT1, TB2086_SMD:SW_SPDT_PCM12, symbol Switch:SW_SPDT
- J2: renamed from J1; footprint TB2086_SMD:Molex_Pico-EZmate_78171-0002_1x02-1MP_P1.20mm_Vertical_rev -> TB2086_SMD:JST_PH_S2B-PH-SM4-TB_1x02-1MP_P2.00mm_Horizontal_rev
- LOGO1: value Logo_Open_Hardware_Small -> Logo_Open_ErgoGen
- S16, S17: value SW_MX_HS -> SW_CHOC_HS; footprint TB2086_KEYSWITCH:SW_MX_HS_1u_reversible -> TB2086_KEYSWITCH:SW_choc_v1_v2_HS_1u_reversible
- S18: value SW_MX_HS -> SW_CHOC_HS; footprint TB2086_KEYSWITCH:SW_MX_HS_1.5u_reversible -> TB2086_KEYSWITCH:SW_choc_v1_v2_HS_1u_reversible
- SW_SPDT2: renamed from SW_SPDT1; value SW_SPDT -> SW_SPDT2; footprint TB2086_SMD:SW_SPDT_PCM12_reversible -> TB2086_SMD:SW_SPDT_PCM12
Connections:
- net BAT: now also SW_SPDT2.3 (C), J3.2 (Pin_2), SW_SPDT1.1 (A); no longer SW_SPDT2.1 (A)
- net GND: now also J1.A12 (GND), J1.B12 (GND), J1.S1 (SHIELD), J3.1 (Pin_1)
- net VCC: now also J1.A9 (VBUS), J1.B9 (VBUS)
- net at J2.2 (Pin_2), SW_SPDT2.2 (B): now also SW_SPDT1.2 (B)
- net at LED3.1 (K), LED4.1 (K): now also J4.3 (Pin_3)
- net at LED1.2 (A), LED2.2 (A), LED3.2 (A)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: now also J4.2 (Pin_2)
- net at LED1.1 (K), LED2.1 (K): now also J4.1 (Pin_1)
- net at JP3.2 (B): now also J1.A5 (CC1)
- net at JP2.2 (C): now also J1.B5 (CC2)
- no-connect marks 8 -> 9
Other:
- moved on the sheet: D10, D11, D12, D13, D14, D15, D4, D5, D6, D7, D8, D9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

Commit message: Quick fixes (#16)
* fix version

* updated PCB
Other:
- title: uniCorne Cherry -> VOID 3x5 Hybrid MX
Changed lines of the file:
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@@
 	(paper "A3")
 	(title_block
-		(title "uniCorne Cherry")
-		(date "2023-07-20")
-		(rev "0.9")
+		(title "VOID 3x5 Hybrid MX")
+		(date "2025-02-02")
+		(rev "0.6.1")
 		(company "Thunderbird2086")
 	)

Commit message: updated kicad data
Parts:
- R1, R2: footprint Resistor_SMD:R_0805_2012Metric_Pad1.20x1.40mm_HandSolder -> TB2086_SMD:R_0805_2012Metric_Pad1.20x1.40mm_HandSolder
- S18: footprint TB2086_KEYSWITCH:SW_choc_v1_v2_HS_1u_reversible -> TB2086_KEYSWITCH:SW_choc_v1_v2_HS_1.5u_reversible
Changed lines of the file:
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@@
 			)
 		)
-		(property "Footprint" "Resistor_SMD:R_0805_2012Metric_Pad1.20x1.40mm_HandSolder"
+		(property "Footprint" "TB2086_SMD:R_0805_2012Metric_Pad1.20x1.40mm_HandSolder"
 			(at 67.31 77.978 90)
 			(effects
@@
 			)
 		)
-		(property "Footprint" "Resistor_SMD:R_0805_2012Metric_Pad1.20x1.40mm_HandSolder"
+		(property "Footprint" "TB2086_SMD:R_0805_2012Metric_Pad1.20x1.40mm_HandSolder"
 			(at 67.31 68.707 90)
 			(effects
@@
 			)
 		)
-		(property "Footprint" "TB2086_KEYSWITCH:SW_choc_v1_v2_HS_1u_reversible"
+		(property "Footprint" "TB2086_KEYSWITCH:SW_choc_v1_v2_HS_1.5u_reversible"
 			(at 188.976 105.664 0)
 			(effects
